File: LineSense.brd (EAGLE design)
At the start: 100 x 45 mm, 48 parts, among them IC1 NJM2904M-TE1, IC2 NE555D, J1 1744426-4, Q1 SFH_3410-1_2-Z, Q2 2SC2712-GR,LF, Q3 2SC2712-GR,LF, Q4 2SC2712-GR,LF, Q5 2SC2712-GR,LF, Q6 2SC2712-GR,LF

Commit message: The First ver2.x
Parts:
- removed D1: PMEG6010CEGWX, SamacSys_Parts:PMEG6010CEGWX
- removed J1: 1744426-4, SamacSys_Parts:17444264
- removed L1: CBC2518T470K, SamacSys_Parts:INDC2518X200N
- removed Q2: 2SC2712-GR,LF, SamacSys_Parts:SSM3J334RLF
- added C9: 220n, rcl:C0603
- added CN1: (no value), jst-xh:S3B-XH-A
- added IC3: NJM2904M, SamacSys_Parts:SOIC127P680X200-8N
- added R18: 0, rcl:R0603
- C1: value 560n -> 15n
- C12: value EEE-HA1E220P -> 10u; device SamacSys_Parts:EEE1AA101SP -> rcl:C1210
- C2: value 2.7n -> 100n
- C5: value 100n -> 6.8n
- C8: value EEE-HA1E220P -> 4.7u; device SamacSys_Parts:EEE1AA101SP -> rcl:C1210
- IC1: value NJM2904M-TE1 -> NJM78L05UA-TE1; device SamacSys_Parts:SOP65P400X100-8N -> SamacSys_Parts:SOT-89-3
- R14: value 13k -> 1.5k
- R15: value 15k -> 2.7k
- R16: value 10k -> 100k
- R3: value 68 -> 10k; device rcl:R2512 -> rcl:R0603
- R7: value 10k -> 56k
- moved C11 36.3 mm to (24.2, 13.6), turned to 90 degrees
- moved R7 32.4 mm to (69.9, 30.7), turned to 270 degrees
- moved IC1 10.1 mm to (46.6, 11.4), turned to 90 degrees
- moved C12 9.74 mm to (81.9, 16.6), turned to 270 degrees
- moved C1 8.05 mm to (44.7, 21.0), turned to 270 degrees
- moved R3 6.10 mm to (41.5, 21.0), turned to 90 degrees
- moved R17 4.34 mm to (76.7, 18.0), turned to 0 degrees
- moved TP3 3.79 mm to (32.6, 21.8)
- moved C8 3.05 mm to (59.8, 10.1)
- moved TP4 2.42 mm to (47.8, 20.0)
- moved TP1 2.41 mm to (74.6, 16.0)
- moved C7 2.34 mm to (59.9, 31.5)
- moved C13 2.16 mm to (84.8, 17.3), turned to 270 degrees
- moved LED1 2.05 mm to (87.9, 16.7), turned to 270 degrees
- moved TP5 1.80 mm to (54.3, 32.1)
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Connections:
- removed net N$14: C1.2, D1.2, L1.1, R3.1, TP4.TP
- removed net N$3: Q2.1, R7.1
- new net +5V: C11.1, IC1.1, Q1.3
- net +12V: now also C9.1, CN1.3, IC1.3, IC3.8; no longer C11.1, IC1.8, J1.1, Q1.3, Q2.3
- net AMP_IN: now also C1.2, IC3.5, R3.1, TP4.TP; no longer D1.1, IC1.5
- net GND: now also C9.2, CN1.1, IC1.2, IC3.4; no longer J1.4, L1.2
- net N$17: now also R7.2
- net N$19: now also R7.1
- net N$2: now also Q3.2, R18.1, R8.2; no longer IC1.1, R7.2
- net N$6: now also IC3.2; no longer IC1.2
- net N$7: now also IC3.7; no longer IC1.7
- net PREAMP_IN: now also IC3.3; no longer IC1.3
- net PREAMP_OUT: now also IC3.1; no longer Q2.2
- net SIG_OUT: now also CN1.2, IC3.6, R18.2; no longer IC1.6, J1.2, Q3.2, R8.2
Routing:
- net +12V: track 137.5 -> 108.8 mm
- net +5V: track 0.00 -> 28.5 mm
- net N$14: track 19.0 -> 0.00 mm
- net N$3: track 18.1 -> 0.00 mm
- net SIG_OUT: track 63.2 -> 46.2 mm, vias 4 -> 0
- net N$2: track 3.32 -> 17.4 mm
- net N$17: track 37.2 -> 27.2 mm, vias 2 -> 0
- net PREAMP_OUT: track 20.3 -> 11.2 mm
- net N$19: track 4.80 -> 9.64 mm
- net N$16: track 7.35 -> 2.66 mm
- net AMP_IN: track 15.2 -> 19.4 mm
- net N$8: track 23.6 -> 20.9 mm
- net LED_OUT: track 8.45 -> 5.84 mm
- net PREAMP_IN: track 17.5 -> 16.1 mm
- net N$5: track 13.7 -> 14.6 mm
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- removed copper zone on layer 1, net N$9
Other:
- outline, holes or cut-outs redrawn
- board text added: "Line Sense v2.0"

Commit message: Update load resistance of reciever
Parts:
- R1: value 500k -> 100k
Changed lines of the file:
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@@
 <attribute name="VALUE" x="87.836" y="9.306" size="1.27" layer="27" align="center"/>
 </element>
-<element name="R1" library="rcl" library_urn="urn:adsk.eagle:library:334" package="R0603" package3d_urn="urn:adsk.eagle:package:23555/3" value="500k" x="23.2918" y="27.432" smashed="yes" rot="R270">
+<element name="R1" library="rcl" library_urn="urn:adsk.eagle:library:334" package="R0603" package3d_urn="urn:adsk.eagle:package:23555/3" value="100k" x="23.2918" y="27.432" smashed="yes" rot="R270">
 <attribute name="NAME" x="21.2268" y="29.067" size="1.27" layer="25" rot="R270"/>
 <attribute name="POPULARITY" value="70" x="-17.3482" y="-3.048" size="1.778" layer="27" rot="R270" display="off"/>
