File: LineSense.brd (EAGLE design)
At the start: 100 x 45 mm, 45 parts, among them IC1 NJM2904M-TE1, IC2 NE555D, J1 1744426-4, Q1 SFH_3410-1_2-Z, Q2 2SC2712-GR,LF, Q3 2SC2712-GR,LF, Q5 2SC2712-GR,LF, Q6 2SC2712-GR,LF

Commit message: modify
Parts:
- R13: value 4.7k -> 2.2k
Changed lines of the file:
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@@
 <attribute name="VALUE" x="90.691" y="3.11" size="1.27" layer="27" rot="R90"/>
 </element>
-<element name="R13" library="rcl" library_urn="urn:adsk.eagle:library:334" package="R0603" package3d_urn="urn:adsk.eagle:package:23555/3" value="4.7k" x="71.986" y="14.402" smashed="yes" rot="R90">
+<element name="R13" library="rcl" library_urn="urn:adsk.eagle:library:334" package="R0603" package3d_urn="urn:adsk.eagle:package:23555/3" value="2.2k" x="71.986" y="14.402" smashed="yes" rot="R90">
 <attribute name="NAME" x="71.351" y="13.767" size="1.27" layer="25" rot="R90"/>
 <attribute name="POPULARITY" value="70" x="112.626" y="71.552" size="1.778" layer="27" rot="R90" display="off"/>
