File: LineSense.sch (EAGLE design)
At the start: 48 parts, among them IC1 NJM78L05UA-TE1, IC2 NE555D, IC3 NJM2904M, Q1 SFH_3410-1_2-Z, Q3 2SC2712-GR,LF, Q4 2SC2712-GR,LF, Q5 2SC2712-GR,LF, Q6 2SC2712-GR,LF

Commit message: Update load resistance of reciever
Parts:
- R1: value 500k -> 100k
Changed lines of the file:
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@@
 </classes>
 <parts>
-<part name="R1" library="rcl" library_urn="urn:adsk.eagle:library:334" deviceset="R-EU_" device="R0603" package3d_urn="urn:adsk.eagle:package:23555/3" value="500k"/>
+<part name="R1" library="rcl" library_urn="urn:adsk.eagle:library:334" deviceset="R-EU_" device="R0603" package3d_urn="urn:adsk.eagle:package:23555/3" value="100k"/>
 <part name="R4" library="rcl" library_urn="urn:adsk.eagle:library:334" deviceset="R-EU_" device="R0603" package3d_urn="urn:adsk.eagle:package:23555/3" value="2.2k"/>
 <part name="R5" library="rcl" library_urn="urn:adsk.eagle:library:334" deviceset="R-TRIMM" device="3339P" package3d_urn="urn:adsk.eagle:package:23757/1" value="100k"/>
