File: LineSense.sch (EAGLE design)
At the start: 48 parts, among them IC1 NJM2904M-TE1, IC2 NE555D, J1 1744426-4, Q1 SFH_3410-1_2-Z, Q2 2SC2712-GR,LF, Q3 2SC2712-GR,LF, Q4 2SC2712-GR,LF, Q5 2SC2712-GR,LF, Q6 2SC2712-GR,LF

Commit message: v1.2
Parts:
- removed Q4: 2SC2712-GR,LF, SamacSys_Parts:2SC2712-GR,LF
- removed R8: 3.6k, rcl:R-EU_R0603
- removed R9: 620, rcl:R-EU_R0603
- R1: value 500k -> 560k
- R13: value 7.5k -> 4.7k
- R2, R7: value 10k -> 0
Connections:
- net +12V renamed +5V
- removed net N$10: Q4.B, R8.1, R9.2
- net GND: no longer Q4.E, R9.1
- net N$8: no longer Q4.C
- net SIG_OUT: no longer R8.2

Commit message: modify
Parts:
- R13: value 4.7k -> 2.2k
Changed lines of the file:
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@@
 <part name="Q5" library="SamacSys_Parts" deviceset="2SC2712-GR,LF" device=""/>
 <part name="Q6" library="SamacSys_Parts" deviceset="2SC2712-GR,LF" device=""/>
-<part name="R13" library="rcl" library_urn="urn:adsk.eagle:library:334" deviceset="R-EU_" device="R0603" package3d_urn="urn:adsk.eagle:package:23555/3" value="4.7k"/>
+<part name="R13" library="rcl" library_urn="urn:adsk.eagle:library:334" deviceset="R-EU_" device="R0603" package3d_urn="urn:adsk.eagle:package:23555/3" value="2.2k"/>
 <part name="LED1" library="SamacSys_Parts" deviceset="XZCB25X109FS" device=""/>
 <part name="IC2" library="SamacSys_Parts" deviceset="NE555D" device=""/>
